Commit message: Ex classes updated

File: Aula12/p_spombinho_description/urdf/p_spombinho.gazebo.xacro (robot description, xacro)
@@ -1,4 +1,6 @@
 <?xml version="1.0"?>
-<robot name="turtlebot3_waffle_pi_sim" xmlns:xacro="http://ros.org/wiki/xacro">
+<robot name="s_pombinho_sim" xmlns:xacro="http://ros.org/wiki/xacro">
+<!--  <xacro:arg name="player_name" default="p_spombinho"/>-->
+<!--  <xacro:arg name="player_color" default="Blue"/>-->
   <xacro:arg name="laser_visual"  default="false"/>
   <xacro:arg name="camera_visual" default="false"/>
@@ -15,4 +17,5 @@
     <maxVel>0.1</maxVel>
     <fdir1>1 0 0</fdir1>
+<!--    <material>Gazebo/${player_color}</material>-->
     <material>Gazebo/Blue</material>
   </gazebo>
@@ -25,4 +28,5 @@
     <maxVel>0.1</maxVel>
     <fdir1>1 0 0</fdir1>
+<!--    <material>Gazebo/${player_color}</material>-->
     <material>Gazebo/Blue</material>
   </gazebo>

File: Aula12/p_spombinho_description/urdf/p_spombinho.urdf.xacro (robot description, xacro)
@@ -1,6 +1,18 @@
 <?xml version="1.0" ?>
-<robot name="turtlebot3_waffle_pi" xmlns:xacro="http://ros.org/wiki/xacro">
+<robot name="p_spombinho" xmlns:xacro="http://ros.org/wiki/xacro">
   <xacro:include filename="$(find turtlebot3_description)/urdf/common_properties.xacro"/>
   <xacro:include filename="$(find p_spombinho_description)/urdf/p_spombinho.gazebo.xacro"/>
+  <!--Args are local, properties are global, so we copy the values of the arguments to the properties-->
+  <xacro:arg name="player_name" default="s_pombinho" />
+  <xacro:arg name="player_color" default="Orange" /> <!-- e.g. Red, Orange. Must exist in Gazebo/Colors and be defined in properties.xacro.-->
+  <!--Properties are global so they can be viewed from inside the included xacros-->
+  <!--  args are used with $(arg arg_name), properties are used as ${property_name}-->
+  <xacro:property name="player_name" value="$(arg player_name)"/>
+  <xacro:property name="player_color" value="$(arg player_color)"/>
+  <!-- Include other files-->
+<!--  <xacro:include filename="$(find p_spombinho_description)/urdf/properties.xacro"/>-->
+  <!--  <xacro:include filename="$(find p_spombinho_description)/urdf/player.gazebo.xacro"/>-->
+  <xacro:include filename="$(find ${player_name}_description)/urdf/player.gazebo.macro.xacro"/>
+  <xacro:gazebo_macro player_color="${player_color}" laser_visual="true" camera_visual="false" imu_visual="true"/>
   <link name="base_footprint"/>
   <joint name="base_joint" type="fixed">
@@ -43,5 +55,5 @@
         <mesh filename="package://turtlebot3_description/meshes/wheels/left_tire.stl" scale="0.001 0.001 0.001"/>
       </geometry>
-      <material name="dark"/>
+      <material name="blue"/>
     </visual>
     <collision>
@@ -71,5 +83,5 @@
         <mesh filename="package://turtlebot3_description/meshes/wheels/right_tire.stl" scale="0.001 0.001 0.001"/>
       </geometry>
-      <material name="dark"/>
+      <material name="blue"/>
     </visual>
     <collision>

Commit message: Ex classes updated

File: Aula12/p_spombinho_description/urdf/p_spombinho.gazebo.xacro (robot description, xacro)
@@ -1,6 +1,4 @@
 <?xml version="1.0"?>
 <robot name="s_pombinho_sim" xmlns:xacro="http://ros.org/wiki/xacro">
-<!--  <xacro:arg name="player_name" default="p_spombinho"/>-->
-<!--  <xacro:arg name="player_color" default="Blue"/>-->
   <xacro:arg name="laser_visual"  default="false"/>
   <xacro:arg name="camera_visual" default="false"/>
@@ -17,5 +15,5 @@
     <maxVel>0.1</maxVel>
     <fdir1>1 0 0</fdir1>
-<!--    <material>Gazebo/${player_color}</material>-->
+    <material>Gazebo/${player_color}</material>
     <material>Gazebo/Blue</material>
   </gazebo>

File: Aula12/p_spombinho_description/urdf/p_spombinho.urdf.xacro (robot description, xacro)
@@ -2,5 +2,5 @@
 <robot name="p_spombinho" xmlns:xacro="http://ros.org/wiki/xacro">
   <xacro:include filename="$(find turtlebot3_description)/urdf/common_properties.xacro"/>
-  <xacro:include filename="$(find p_spombinho_description)/urdf/p_spombinho.gazebo.xacro"/>
+<!--  <xacro:include filename="$(find p_spombinho_description)/urdf/p_spombinho.gazebo.xacro"/>-->
   <!--Args are local, properties are global, so we copy the values of the arguments to the properties-->
   <xacro:arg name="player_name" default="s_pombinho" />
@@ -11,7 +11,5 @@
   <xacro:property name="player_color" value="$(arg player_color)"/>
   <!-- Include other files-->
-<!--  <xacro:include filename="$(find p_spombinho_description)/urdf/properties.xacro"/>-->
-  <!--  <xacro:include filename="$(find p_spombinho_description)/urdf/player.gazebo.xacro"/>-->
-  <xacro:include filename="$(find ${player_name}_description)/urdf/player.gazebo.macro.xacro"/>
+  <xacro:include filename="$(find p_spombinho_description)/urdf/p_spombinho.gazebo.macro.xacro"/>
   <xacro:gazebo_macro player_color="${player_color}" laser_visual="true" camera_visual="false" imu_visual="true"/>
   <link name="base_footprint"/>

Commit message: Ex classes updated

File: Aula12/p_spombinho_description/urdf/p_spombinho.gazebo.xacro (robot description, xacro)
@@ -15,5 +15,5 @@
     <maxVel>0.1</maxVel>
     <fdir1>1 0 0</fdir1>
-    <material>Gazebo/${player_color}</material>
+<!--    <material>Gazebo/${player_color}</material>-->
     <material>Gazebo/Blue</material>
   </gazebo>

File: Aula12/p_spombinho_description/urdf/p_spombinho.urdf.xacro (robot description, xacro)
@@ -5,5 +5,6 @@
   <!--Args are local, properties are global, so we copy the values of the arguments to the properties-->
   <xacro:arg name="player_name" default="s_pombinho" />
-  <xacro:arg name="player_color" default="Orange" /> <!-- e.g. Red, Orange. Must exist in Gazebo/Colors and be defined in properties.xacro.-->
+  <xacro:arg name="player_color" default="Orange" />
+  <!-- e.g. Red, Orange. Must exist in Gazebo/Colors and be defined in properties.xacro.-->
   <!--Properties are global so they can be viewed from inside the included xacros-->
   <!--  args are used with $(arg arg_name), properties are used as ${property_name}-->
@@ -12,5 +13,6 @@
   <!-- Include other files-->
   <xacro:include filename="$(find p_spombinho_description)/urdf/p_spombinho.gazebo.macro.xacro"/>
-  <xacro:gazebo_macro player_color="${player_color}" laser_visual="true" camera_visual="false" imu_visual="true"/>
+  <xacro:gazebo_macro player_color="${player_color}" laser_visual="false" camera_visual="false" imu_visual="false"/>
+<!--  <xacro:gazebo_macro player_color="${player_color}" />-->
   <link name="base_footprint"/>
   <joint name="base_joint" type="fixed">
