Commit message: professor th added

File: Aula12/p_spombinho_description/urdf/p_spombinho.gazebo.macro.xacro (robot description, xacro)
@@ -7,5 +7,18 @@
 <!--  <xacro:arg name="imu_visual"    default="false"/>-->
   <gazebo reference="base_link">
-    <material>Gazebo/DarkGrey</material>
+    <material>Gazebo/${player_color}</material>
+  </gazebo>
+  <gazebo reference="base_link">
+    <sensor name="base_link" type="contact">
+      <update_rate>1000.0</update_rate>
+      <always_on>true</always_on>
+      <contact>
+        <collision>base_footprint_fixed_joint_lump__base_link_collision_collision</collision>
+      </contact>
+      <plugin name="base_link_contact_sensor_plugin" filename="libgazebo_ros_bumper.so">
+        <bumperTopicName>contact</bumperTopicName>
+        <frameName>world</frameName>
+      </plugin>
+    </sensor>
   </gazebo>
   <gazebo reference="wheel_left_link">
@@ -17,6 +30,6 @@
     <maxVel>0.1</maxVel>
     <fdir1>1 0 0</fdir1>
-    <material>Gazebo/${player_color}</material>
-<!--    <material>Gazebo/Blue</material>-->
+<!--    <material>Gazebo/${player_color}</material>-->
+    <material>Gazebo/FlatBlack</material>
   </gazebo>
   <gazebo reference="wheel_right_link">
@@ -28,6 +41,6 @@
     <maxVel>0.1</maxVel>
     <fdir1>1 0 0</fdir1>
-    <material>Gazebo/${player_color}</material>
-<!--    <material>Gazebo/Blue</material>-->
+<!--    <material>Gazebo/${player_color}</material>-->
+    <material>Gazebo/FlatBlack</material>
   </gazebo>
   <gazebo reference="caster_back_right_link">
