Commit message: professor th added

File: Aula12/p_spombinho_description_class/urdf/p_spombinho.gazebo.macro.xacro (robot description, xacro)
@@ -14,5 +14,5 @@
       <always_on>true</always_on>
       <contact>
-        <collision>base_footprint_fixed_joint_lump__base_link_collision_collision</collision>
+        <collision>"base_footprint_fixed_joint_lump__base_link_collision"</collision>
       </contact>
       <plugin name="base_link_contact_sensor_plugin" filename="libgazebo_ros_bumper.so">
